Commit message: URDF Updated

File: description/depth_camera.xacro (robot description, xacro)
@@ -4,5 +4,5 @@
         <parent link = "chassis" />
         <child link = "camera_link" />
-        <origin xyz = "0.375 0 0.15" rpy = "0 0 0" />
+        <origin xyz = "0.375 0 0.08" rpy = "0 0 0" />
     </joint>
     <link name = "camera_link" >
@@ -23,5 +23,5 @@
     <gazebo reference="camera_link">
         <material>Gazebo/Black</material>
-        <sensor name="camera" type="camera"> <!-- lidar sensor -->
+        <sensor name="camera" type="depth"> <!-- lidar sensor -->
             <pose> 0 0 0 0 0 0 </pose>   <!-- origin of sensor -->
             <visualize>true</visualize>
@@ -30,5 +30,5 @@
               <horizontal_fov>1.089</horizontal_fov>  <!-- hortizontal field of view-->
               <image>
-                <format>R8g8b8</format>
+                <format>B8G8R8</format>
                 <width>640</width>
                 <height>480</height>
@@ -42,4 +42,6 @@
             <plugin name="camera_controller" filename="libgazebo_ros_camera.so">
                 <frame_name>camera_link_optical</frame_name>
+                <min_depth>0.1</min_depth>
+                <max_depth>100</max_depth>
             </plugin>
         </sensor>

File: description/lidar.xacro (robot description, xacro)
@@ -4,5 +4,5 @@
         <parent link = "chassis" />
         <child link = "laser_frame" />
-        <origin xyz = "0.05 0 0.130" rpy = "0 0 0" />
+        <origin xyz = "0.05 0 0.2" rpy = "0 0 0" />
     </joint>
     <link name = "laser_frame" >
@@ -11,5 +11,5 @@
          <cylinder radius = "0.04" length = "0.04" />
        </geometry>
-       <material name = "red" />
+       <material name = "blue" />
      </visual>
      <collision>
@@ -24,5 +24,5 @@
     </link>
     <gazebo reference="laser_frame">
-        <material>Gazebo/Red</material>
+        <material>Gazebo/Blue</material>
         <sensor name="laser" type="ray"> <!-- lidar sensor -->
             <pose> 0 0 0 0 0 0 </pose>   <!-- origin of sensor -->

File: description/robot.urdf.xacro (robot description, xacro)
@@ -2,6 +2,8 @@
 <robot xmlns:xacro="http://www.ros.org/wiki/xacro"  name="robot">
     <xacro:include filename = "robot_core.xacro" />
-    <xacro:include filename = "gazebo_control.xacro" />
+   <!-- <xacro:include filename = "gazebo_control.xacro" /> -->
+    <xacro:include filename = "ros2_control.xacro" />
     <xacro:include filename = "lidar.xacro" />
     <xacro:include filename = "camera.xacro" />
+    <!-- <xacro:include filename = "depth_camera.xacro" /> -->
 </robot>

File: description/robot_core.xacro (robot description, xacro)
@@ -1,132 +1,193 @@
 <?xml version="1.0"?>
-<robot xmlns:xacro="http://www.ros.org/wiki/xacro" >
-<xacro:include filename = "inertial_macros.xacro" />
-<material name = "white">
-<color rgba = "1 1 1 1" />
-</material>
-<material name = "orange">
-<color rgba = "1 0.3 0.1 1" />
-</material>
-<material name = "blue">
-<color rgba = "0.2 0.2 1 1" />
-</material>
-<material name = "black">
-<color rgba = "0 0 0 1" />
-</material>
-<material name = "red">
-<color rgba = "1 0 0 1" />
-</material>
-<!-- BASE LINK -->
-<link name = "base_link">
-</link>
-<!-- CHASSIS LINK -->
-<joint name = "chassis_joint" type = "fixed" >
-        <parent link = "base_link" />
-        <child link = "chassis" />
-        <origin xyz = "-0.1 0 0" />
-</joint>
-<link name = "chassis">
-    <visual>
-        <origin xyz = "0.135 0 0.05" /> <!--origin point-->
-        <geometry>
-            <box size = "0.368 0.257 0.137" /> <!--chassis dimensions(meters)-->
-        </geometry>
-        <material name = "white" />
-    </visual>
-    <collision>
-        <origin xyz = "0.135 0 0.05" /> <!--origin point-->
-        <geometry>
-            <box size = "0.368 0.257 0.137" /> <!--chassis dimensions(meters)-->
-        </geometry>
-    </collision>
-    <!-- moment of interia -->
-    <xacro:inertial_box mass = "0.5" x = "0.368" y = "0.257" z = "0.137" >
-       <origin xyz = "0.184 0 0.0685" rpy = "0 0 0"/>
-    </xacro:inertial_box>
-</link>
-<gazebo reference = "chassis">
-     <material>Gazebo/White</material>
-</gazebo>
-<!-- LEFT WHEEL LINK-->
-<joint name = "left_wheel_joint" type = "continuous">
-     <parent link = "base_link" />
-     <child link = "left_wheel" />
-     <origin xyz = "-0.08 0.14 -0.015" rpy = "-${pi/2} 0 0" />
-     <axis xyz = "0 0 1" />
-</joint>
-<link name = "left_wheel">
-    <visual>
-         <geometry>
-              <cylinder radius = "0.04" length = "0.02" />
-         </geometry>
-         <material name = "blue" />
-    </visual>
-    <collision>
-         <geometry>
-              <cylinder radius = "0.04" length = "0.02" />
-         </geometry>
-    </collision>
-    <!-- moment of inertia -->
-    <xacro:inertial_cylinder mass = "0.2" length = "0.02" radius = "0.04" >
-      <origin xyz = "0 0 0" rpy = "0 0 0" />
-    </xacro:inertial_cylinder>
-</link>
-<gazebo reference = "left_wheel">
-     <material>Gazebo/Blue</material>
-</gazebo>
-<!-- RIGHT WHEEL LINK-->
-<joint name = "right_wheel_joint" type = "continuous">
-     <parent link = "base_link" />
-     <child link = "right_wheel" />
-     <origin xyz = "-0.08 -0.14 -0.015" rpy = "${pi/2} 0 0" /> <!-- -0.175m from origin in y,roll,pitch,yaw-->
-     <axis xyz = "0 0 -1" />
-</joint>
-<link name = "right_wheel">
-    <visual>
-         <geometry>
-              <cylinder radius = "0.04" length = "0.02" />
-         </geometry>
-         <material name = "blue" />
-    </visual>
-    <collision>
-         <geometry>
-              <cylinder radius = "0.04" length = "0.02" />
-         </geometry>
-    </collision>
-    <!-- moment of inertia-->
-    <xacro:inertial_cylinder mass = "0.2" length = "0.02" radius = "0.04" >
-    <origin xyz = "0 0 0" rpy = "0 0 0" />
-    </xacro:inertial_cylinder>
-</link>
-<gazebo reference = "right_wheel">
-     <material>Gazebo/Blue</material>
-</gazebo>
-<!-- CASTER WHEEL LINK -->
-<joint name = "caster_wheel_joint" type="fixed">
-    <parent link = "chassis" />
-    <child link = "caster_wheel" />
-    <origin xyz = "0.27 0 -0.015" rpy = "0 0 0"/>
-</joint>
-<link name = "caster_wheel" >
+<robot xmlns:xacro="http://www.ros.org/wiki/xacro">
+     <xacro:include filename="inertial_macros.xacro" />
+     <xacro:property name="chassis_length" value="0.368" />
+     <xacro:property name="chassis_width" value="0.257" />
+     <xacro:property name="chassis_height" value="0.137" />
+     <xacro:property name="chassis_mass" value="2.1" />
+     <!--robot_mass = [my_mass + robot_mass_unknown] - my_mass = 61.4 - 59.3 = 2.1kg-->
+     <xacro:property name="wheel_radius" value="0.033" />
+     <xacro:property name="wheel_thickness" value="0.026" />
+     <xacro:property name="wheel_mass" value="0.038" />
+     <xacro:property name="wheel_offset_x" value="0.103" />
+     <xacro:property name="wheel_offset_y" value="0.145" />
+     <xacro:property name="wheel_offset_z" value="-0.032" />
+     <xacro:property name="caster_wheel_radius" value="0.025" />
+     <xacro:property name="caster_wheel_mass" value="0.032" />
+     <xacro:property name="caster_wheel_offset_x" value="0.323" />
+     <xacro:property name="caster_wheel_offset_z" value="${wheel_offset_z - wheel_radius + caster_wheel_radius}" />
+     <material name="white">
+          <color rgba="1 1 1 1" />
+     </material>
+     <material name="orange">
+          <color rgba="1 0.3 0.1 1" />
+     </material>
+     <material name="blue">
+          <color rgba="0.2 0.2 1 1" />
+     </material>
+     <material name="black">
+          <color rgba="0 0 0 1" />
+     </material>
+     <material name="red">
+          <color rgba="1 0 0 1" />
+     </material>
+     <!-- BASE LINK -->
+     <link name="base_link">
+     </link>
+     <!-- CHASSIS LINK -->
+     <joint name="chassis_joint" type="fixed">
+          <parent link="base_link" />
+          <child link="chassis" />
+          <origin xyz="${-wheel_offset_x} 0 ${-wheel_offset_z}" />
+     </joint>
+     <link name="chassis">
      <visual>
-       <geometry>
-         <sphere radius = "0.04" />
-       </geometry>
-       <material name = "black" />
+          <origin xyz="${chassis_length/2} 0 ${chassis_height/2}" />
+          <geometry>
+               <box size="${chassis_length} ${chassis_width} ${chassis_height}" />
+          </geometry>
+          <material name="white" />
      </visual>
      <collision>
-       <geometry>
-         <sphere radius = "0.04" />
-       </geometry>
+          <origin xyz="${chassis_length/2} 0 ${chassis_height/2}" />
+          <geometry>
+               <box size="${chassis_length} ${chassis_width} ${chassis_height}" />
+          </geometry>
      </collision>
-     <!-- moment of inertia -->
-     <xacro:inertial_sphere mass = "0.2" radius = "0.04" >
-     <origin xyz = "0 0 0" rpy = "0 0 0" />
+     <xacro:inertial_box mass="0.5" x="${chassis_length}" y="${chassis_width}" z="${chassis_height}">
+          <origin xyz="${chassis_length/2} 0 ${chassis_height/2}" rpy="0 0 0" />
+     </xacro:inertial_box>
+     </link>
+     <gazebo reference="chassis">
+          <material>Gazebo/White</material>
+     </gazebo>
+     <!-- LEFT WHEEL LINK -->
+     <joint name="left_wheel_joint" type="continuous">
+          <parent link="base_link" />
+          <child link="left_wheel" />
+          <origin xyz="0 ${wheel_offset_y} 0" rpy="-${pi/2} 0 0" />
+          <axis xyz="0 0 1" />
+     </joint>
+     <link name="left_wheel">
+     <visual>
+          <geometry>
+               <cylinder radius="${wheel_radius}" length="${wheel_thickness}" />
+          </geometry>
+          <material name="blue" />
+     </visual>
+     <collision>
+          <geometry>
+               <sphere radius="${wheel_radius}" />
+          </geometry>
+     </collision>
+     <xacro:inertial_cylinder mass="${wheel_mass}" length="${wheel_thickness}" radius="${wheel_radius}">
+          <origin xyz="0 0 0" rpy="0 0 0" />
+     </xacro:inertial_cylinder>
+     </link>
+     <gazebo reference="left_wheel">
+          <material>Gazebo/Blue</material>
+     </gazebo>
+     <!-- RIGHT WHEEL LINK -->
+     <joint name="right_wheel_joint" type="continuous">
+          <parent link="base_link" />
+          <child link="right_wheel" />
+          <origin xyz="0 ${-wheel_offset_y} 0" rpy="${pi/2} 0 0" />
+          <axis xyz="0 0 -1" />
+     </joint>
+     <link name="right_wheel">
+     <visual>
+          <geometry>
+               <cylinder radius="${wheel_radius}" length="${wheel_thickness}" />
+          </geometry>
+          <material name="blue" />
+     </visual>
+     <collision>
+          <geometry>
+               <sphere radius="${wheel_radius}" />
+          </geometry>
+     </collision>
+     <xacro:inertial_cylinder mass="${wheel_mass}" length="${wheel_thickness}" radius="${wheel_radius}">
+          <origin xyz="0 0 0" rpy="0 0 0" />
+     </xacro:inertial_cylinder>
+     </link>
+     <gazebo reference="right_wheel">
+          <material>Gazebo/Blue</material>
+     </gazebo>
+     <!-- CASTER WHEEL LINK -->
+     <joint name="caster_wheel_joint" type="fixed">
+          <parent link="chassis" />
+          <child link="caster_wheel" />
+          <origin xyz="${caster_wheel_offset_x} 0 ${caster_wheel_offset_z}" />
+     </joint>
+     <link name="caster_wheel">
+     <visual>
+          <geometry>
+               <sphere radius="${caster_wheel_radius}" />
+          </geometry>
+          <material name="white" />
+     </visual>
+     <collision>
+          <geometry>
+               <sphere radius="${caster_wheel_radius}" />
+          </geometry>
+     </collision>
+     <xacro:inertial_sphere mass="${caster_wheel_mass}" radius="${caster_wheel_radius}">
+          <origin xyz="0 0 0" rpy="0 0 0" />
      </xacro:inertial_sphere>
-</link>
-<gazebo reference = "caster_wheel">
-     <material>Gazebo/Black</material>
-     <mu1 value = "0.001" />
-     <mu2 value = "0.001" />
-</gazebo>
+     </link>
+     <gazebo reference="caster_wheel">
+          <material>Gazebo/White</material>
+          <mu1 value="0.001" />
+          <mu2 value="0.001" />
+     </gazebo>
+     <!--CASTER WHEEL SUPPORT LINK-->
+     <joint name="caster_wheel_support_joint" type="fixed">
+          <parent link="chassis" />
+          <child link="caster_wheel_support" />
+          <origin xyz="${caster_wheel_offset_x} 0 0" />
+     </joint>
+     <link name="caster_wheel_support">
+     <visual>
+          <geometry>
+               <cylinder radius="${caster_wheel_radius}" length="0.07" />
+          </geometry>
+          <material name="black" />
+     </visual>
+     <collision>
+          <geometry>
+               <cylinder radius="${caster_wheel_radius}" length="0.07" />
+          </geometry>
+     </collision>
+     <xacro:inertial_sphere mass="${caster_wheel_mass}" radius="${caster_wheel_radius}">
+          <origin xyz="0 0 0" rpy="0 0 0" />
+     </xacro:inertial_sphere>
+     </link>
+     <gazebo reference="caster_wheel_support">
+          <material>Gazebo/Black</material>
+     </gazebo>
+     <!--LIDAR SUPPORT LINK-->
+     <joint name="lidar_support_joint" type="fixed">
+          <parent link="chassis" />
+          <child link="lidar_support" />
+          <origin xyz="0.05 0 0.15" />
+     </joint>
+     <link name="lidar_support">
+     <visual>
+          <geometry>
+               <cylinder radius="0.01" length="0.07" />
+          </geometry>
+          <material name="black" />
+     </visual>
+     <collision>
+          <geometry>
+               <cylinder radius="${caster_wheel_radius}" length="0.07" />
+          </geometry>
+     </collision>
+     <xacro:inertial_sphere mass="${caster_wheel_mass}" radius="${caster_wheel_radius}">
+          <origin xyz="0 0 0" rpy="0 0 0" />
+     </xacro:inertial_sphere>
+     </link>
+     <gazebo reference="lidar_support">
+          <material>Gazebo/Black</material>
+     </gazebo>
 </robot>
