Commit message: Added model to Gazebo

File: description/robot.urdf.xacro (robot description, xacro)
@@ -2,3 +2,4 @@
 <robot xmlns:xacro="http://www.ros.org/wiki/xacro"  name="robot">
     <xacro:include filename = "robot_core.xacro" />
+    <xacro:include filename = "gazebo_control.xacro" />
 </robot>

File: description/robot_core.xacro (robot description, xacro)
@@ -31,10 +31,10 @@
         <material name = "white" />
     </visual>
-    <collison>
+    <collision>
         <origin xyz = "0.135 0 0.05" /> <!--origin point-->
         <geometry>
             <box size = "0.368 0.257 0.137" /> <!--chassis dimensions(meters)-->
         </geometry>
-    </collison>
+    </collision>
     <!-- moment of interia -->
     <xacro:inertial_box mass = "0.5" x = "0.368" y = "0.257" z = "0.137" >
@@ -42,4 +42,7 @@
     </xacro:inertial_box>
 </link>
+<gazebo reference = "chassis">
+     <material>Gazebo/White</material>
+</gazebo>
 <!-- LEFT WHEEL LINK-->
 <joint name = "left_wheel_joint" type = "continuous">
@@ -56,9 +59,9 @@
          <material name = "blue" />
     </visual>
-    <collison>
+    <collision>
          <geometry>
               <cylinder radius = "0.04" length = "0.02" />
          </geometry>
-    </collison>
+    </collision>
     <!-- moment of inertia -->
     <xacro:inertial_cylinder mass = "0.1" length = "0.2" radius = "0.04" >
@@ -66,4 +69,7 @@
     </xacro:inertial_cylinder>
 </link>
+<gazebo reference = "left_wheel">
+     <material>Gazebo/Blue</material>
+</gazebo>
 <!-- RIGHT WHEEL LINK-->
 <joint name = "right_wheel_joint" type = "continuous">
@@ -80,9 +86,9 @@
          <material name = "blue" />
     </visual>
-    <collison>
+    <collision>
          <geometry>
               <cylinder radius = "0.04" length = "0.02" />
          </geometry>
-    </collison>
+    </collision>
     <!-- moment of inertia-->
     <xacro:inertial_cylinder mass = "0.1" length = "0.2" radius = "0.04" >
@@ -90,4 +96,7 @@
     </xacro:inertial_cylinder>
 </link>
+<gazebo reference = "right_wheel">
+     <material>Gazebo/Blue</material>
+</gazebo>
 <!-- CASTER WHEEL LINK -->
 <joint name = "caster_wheel_joint" type="fixed">
@@ -103,9 +112,9 @@
        <material name = "black" />
      </visual>
-     <collison>
+     <collision>
        <geometry>
          <cylinder radius = "0.04" length = "0.02" />
        </geometry>
-     </collison>
+     </collision>
      <!-- moment of inertia -->
      <xacro:inertial_cylinder mass = "0.1" length = "0.2" radius = "0.04" >
@@ -113,3 +122,7 @@
      </xacro:inertial_cylinder>
 </link>
+<gazebo reference = "caster_wheel">
+     <material>Gazebo/Black</material>
+     <mu1 value = "0.001" />
+</gazebo>
 </robot>

Commit message: Added Camera

File: description/robot.urdf.xacro (robot description, xacro)
@@ -3,3 +3,5 @@
     <xacro:include filename = "robot_core.xacro" />
     <xacro:include filename = "gazebo_control.xacro" />
+    <xacro:include filename = "lidar.xacro" />
+    <xacro:include filename = "camera.xacro" />
 </robot>

File: description/robot_core.xacro (robot description, xacro)
@@ -13,4 +13,7 @@
 <material name = "black">
 <color rgba = "0 0 0 1" />
+</material>
+<material name = "red">
+<color rgba = "1 0 0 1" />
 </material>
 <!-- BASE LINK -->
@@ -65,5 +68,5 @@
     </collision>
     <!-- moment of inertia -->
-    <xacro:inertial_cylinder mass = "0.1" length = "0.2" radius = "0.04" >
+    <xacro:inertial_cylinder mass = "0.2" length = "0.02" radius = "0.04" >
       <origin xyz = "0 0 0" rpy = "0 0 0" />
     </xacro:inertial_cylinder>
@@ -92,5 +95,5 @@
     </collision>
     <!-- moment of inertia-->
-    <xacro:inertial_cylinder mass = "0.1" length = "0.2" radius = "0.04" >
+    <xacro:inertial_cylinder mass = "0.2" length = "0.02" radius = "0.04" >
     <origin xyz = "0 0 0" rpy = "0 0 0" />
     </xacro:inertial_cylinder>
@@ -103,10 +106,10 @@
     <parent link = "chassis" />
     <child link = "caster_wheel" />
-    <origin xyz = "0.27 0 -0.015" rpy = "-${pi/2} 0 0"/>
+    <origin xyz = "0.27 0 -0.015" rpy = "0 0 0"/>
 </joint>
 <link name = "caster_wheel" >
      <visual>
        <geometry>
-         <cylinder radius = "0.04" length = "0.02" />
+         <sphere radius = "0.04" />
        </geometry>
        <material name = "black" />
@@ -114,15 +117,16 @@
      <collision>
        <geometry>
-         <cylinder radius = "0.04" length = "0.02" />
+         <sphere radius = "0.04" />
        </geometry>
      </collision>
      <!-- moment of inertia -->
-     <xacro:inertial_cylinder mass = "0.1" length = "0.2" radius = "0.04" >
+     <xacro:inertial_sphere mass = "0.2" radius = "0.04" >
      <origin xyz = "0 0 0" rpy = "0 0 0" />
-     </xacro:inertial_cylinder>
+     </xacro:inertial_sphere>
 </link>
 <gazebo reference = "caster_wheel">
      <material>Gazebo/Black</material>
      <mu1 value = "0.001" />
+     <mu2 value = "0.001" />
 </gazebo>
 </robot>

Commit message: Updated Robot Launch File

File: description/robot.urdf.xacro (robot description, xacro)
@@ -1,9 +1,15 @@
 <?xml version="1.0"?>
-<robot xmlns:xacro="http://www.ros.org/wiki/xacro"  name="robot">
-    <xacro:include filename = "robot_core.xacro" />
-   <!-- <xacro:include filename = "gazebo_control.xacro" /> -->
-    <xacro:include filename = "ros2_control.xacro" />
-    <xacro:include filename = "lidar.xacro" />
-    <xacro:include filename = "camera.xacro" />
+<robot xmlns:xacro="http://www.ros.org/wiki/xacro" name="robot">
+    <xacro:arg name="use_ros2_control" default="true" />
+    <xacro:arg name="sim_mode" default="false" />
+    <xacro:include filename="robot_core.xacro" />
+    <xacro:if value="$(arg use_ros2_control)">
+        <xacro:include filename="ros2_control.xacro" />
+    </xacro:if>
+    <xacro:unless value="$(arg use_ros2_control)">
+        <xacro:include filename="gazebo_control.xacro" />
+    </xacro:unless>
+    <xacro:include filename="lidar.xacro" />
+    <xacro:include filename="camera.xacro" />
     <!-- <xacro:include filename = "depth_camera.xacro" /> -->
 </robot>

File: description/ros2_control.xacro (robot description, xacro)
@@ -1,58 +1,61 @@
 <?xml version="1.0"?>
 <robot xmlns:xacro="http://www.ros.org/wiki/xacro" name="robot">
+   <xacro:unless value="$(arg sim_mode)">
       <ros2_control name="VectorBot" type="system">
-      <hardware>
-         <plugin>diffdrive_arduino/DiffDriveArduino</plugin>
-         <param name = "left_wheel_name">left_wheel_joint</param>
-         <param name = "right_wheel_name">right_wheel_joint</param>
-         <param name = "loop_rate">30</param>
-         <param name = "device">/dev/ttyUSB0</param>
-         <param name = "baud_rate">9600</param>
-         <param name = "timeout">1000</param>
-         <param name = "enc_counts_per_rev">889</param>
-      </hardware>
-      <joint name="left_wheel_joint">
-         <command_interface name="velocity">
-            <param name="min">-10</param>
-            <param name="max">-10</param>
-         </command_interface>
-         <state_interface name="velocity" />
-         <state_interface name="position" />
-      </joint>
-      <joint name="right_wheel_joint">
-         <command_interface name="velocity">
-            <param name="min">-10</param>
-            <param name="max">-10</param>
-         </command_interface>
-         <state_interface name="velocity" />
-         <state_interface name="position" />
-      </joint>
-   </ros2_control>
-   <!--
-   <ros2_control name="GazeboSystem" type="system">
-      <hardware>
-         <plugin>gazebo_ros2_control/GazeboSystem</plugin>
-      </hardware>
-      <joint name="left_wheel_joint">
-         <command_interface name="velocity">
-            <param name="min">-10</param>
-            <param name="max">-10</param>
-         </command_interface>
-         <state_interface name="velocity" />
-         <state_interface name="position" />
-      </joint>
-      <joint name="right_wheel_joint">
-         <command_interface name="velocity">
-            <param name="min">-10</param>
-            <param name="max">-10</param>
-         </command_interface>
-         <state_interface name="velocity" />
-         <state_interface name="position" />
-      </joint>
-   </ros2_control>
-   -->
+         <hardware>
+            <plugin>diffdrive_arduino/DiffDriveArduino</plugin>
+            <param name="left_wheel_name">left_wheel_joint</param>
+            <param name="right_wheel_name">right_wheel_joint</param>
+            <param name="loop_rate">30</param>
+            <param name="device">/dev/ttyUSB0</param>
+            <param name="baud_rate">9600</param>
+            <param name="timeout">1000</param>
+            <param name="enc_counts_per_rev">889</param>
+         </hardware>
+         <joint name="left_wheel_joint">
+            <command_interface name="velocity">
+               <param name="min">-10</param>
+               <param name="max">-10</param>
+            </command_interface>
+            <state_interface name="velocity" />
+            <state_interface name="position" />
+         </joint>
+         <joint name="right_wheel_joint">
+            <command_interface name="velocity">
+               <param name="min">-10</param>
+               <param name="max">-10</param>
+            </command_interface>
+            <state_interface name="velocity" />
+            <state_interface name="position" />
+         </joint>
+      </ros2_control>
+   </xacro:unless>
+   <xacro:if value="$(arg sim_mode)">
+      <ros2_control name="GazeboSystem" type="system">
+         <hardware>
+            <plugin>gazebo_ros2_control/GazeboSystem</plugin>
+         </hardware>
+         <joint name="left_wheel_joint">
+            <command_interface name="velocity">
+               <param name="min">-10</param>
+               <param name="max">-10</param>
+            </command_interface>
+            <state_interface name="velocity" />
+            <state_interface name="position" />
+         </joint>
+         <joint name="right_wheel_joint">
+            <command_interface name="velocity">
+               <param name="min">-10</param>
+               <param name="max">-10</param>
+            </command_interface>
+            <state_interface name="velocity" />
+            <state_interface name="position" />
+         </joint>
+      </ros2_control>
+   </xacro:if>
    <gazebo>
-      <plugin name = "gazebo_ros2_control" filename = "libgazebo_ros2_control.so" >
+      <plugin name="gazebo_ros2_control" filename="libgazebo_ros2_control.so">
          <parameters>$(find vector_bot)/config/my_controllers.yaml</parameters>
+         <parameters>$(find vector_bot)/config/gaz_ros2_ctl_use_sim.yaml</parameters>
       </plugin>
    </gazebo>
